Commit message: save env

File: robotis_op_description/robots/robotis_op.urdf (robot description, URDF)
Before this commit: robot robotis_op2, 31 links, 30 joints
Links:
- link MP_ARM_GRIPPER_FIX_DUMMY_L: mass 0.01 -> 0.010
- link MP_ARM_GRIPPER_FIX_DUMMY_R: mass 0.01 -> 0.010
- link MP_ARM_GRIPPER_FIX_L: mass 0.01 -> 0.010
- link MP_ARM_GRIPPER_FIX_R: mass 0.01 -> 0.010
- link MP_ARM_GRIPPER_MOV_L: mass 0.01 -> 0.010
- link MP_ARM_GRIPPER_MOV_R: mass 0.01 -> 0.010
- link MP_ARM_LOW_L: mass 0.01 -> 0.059288504
- link MP_PELVIS_L: mass 0.197 -> 0.167
- link MP_THIGH2_L: mass 0.0070309794 -> 0.11904336
- link MP_TIBIA_L: mass 0.0070309794 -> 0.070309794

File: robotis_op_description/robots/robotis_op.urdf.xacro (robot description, xacro)
@@ -2,4 +2,5 @@
 <robot name="robotis_op2" xmlns:xacro="http://www.ros.org/wiki/xacro">
   <xacro:include filename="$(find robotis_op_description)/robots/robotis_op.urdf.xacro.xml" />
+  <xacro:include filename="$(find robotis_op_description)/urdf/robotis_op.gazebo.xacro" />
   <robotis_op_macro />
 </robot>

File: robotis_op_description/urdf/torso/robotis_op_torso.urdf.xacro (robot description, xacro)
@@ -8,5 +8,5 @@
       <origin xyz="-0.003053 -0.038651 -0.019268" />
       <mass value="0.97559947"/>
-      <inertia ixx="3.1081800"  ixy="-0.25460189"  ixz="2.0318174" iyy="6.3787776" iyz="0.16417863" izz="5.3316425" />
+      <inertia ixx="0.001879411079" ixy="0.0" ixz="0.0" iyy="0.00175933104423" iyz="0.0" izz="0.00181176951575"/>
     </inertial>
     <body_collision_geom_macro />
