Commit message: Create server branch; Fix gzclient not find mesh file problem

File: robotis_op_description/robots/robotis_op_traj.urdf (robot description, URDF)
Before this commit: robot robotis_op2, 31 links, 30 joints
Links:
- link MP_ARM_GRIPPER_FIX_DUMMY_L: mass 0.010 -> 0.01
- link MP_ARM_GRIPPER_FIX_DUMMY_R: mass 0.010 -> 0.01
- link MP_ARM_GRIPPER_FIX_L: mass 0.010 -> 0.01
- link MP_ARM_GRIPPER_FIX_R: mass 0.010 -> 0.01
- link MP_ARM_GRIPPER_MOV_L: mass 0.010 -> 0.01
- link MP_ARM_GRIPPER_MOV_R: mass 0.010 -> 0.01
- link MP_ARM_LOW_L: mass 0.059288504 -> 0.01
- link MP_PELVIS_L: mass 0.167 -> 0.197
- link MP_THIGH2_L: mass 0.11904336 -> 0.0070309794
- link MP_TIBIA_L: mass 0.070309794 -> 0.0070309794
