Commit message: Create server branch; Fix gzclient not find mesh file problem

File: robotis_op_description/robots/robotis_op_norm.urdf (robot description, URDF)
Before this commit: robot robotis_op2, 31 links, 30 joints
Links:
- link MP_ANKLE1_L: geometry collision box size=0.028652 0.08175 0.045; visual mesh filename=file://robotis_op_description/meshes/ankle1_l.STL scale=1 1 1
- link MP_ANKLE1_R: geometry collision box size=0.028652 0.08175 0.045; visual mesh filename=file://robotis_op_description/meshes/ankle1_r.STL scale=1 1 1
- link MP_ANKLE2_L: geometry collision box size=0.008 0.066 0.104; visual mesh filename=file://robotis_op_description/meshes/ankle2_l.STL scale=1 1 1
- link MP_ANKLE2_R: geometry collision box size=0.008 0.066 0.104; visual mesh filename=file://robotis_op_description/meshes/ankle2_r.STL scale=1 1 1
- link MP_ARM_HIGH_L: geometry collision box size=0.06 0.032 0.035; visual mesh filename=file://robotis_op_description/meshes/arm_high_l.STL scale=1 1 1
- link MP_ARM_HIGH_R: geometry collision box size=0.06 0.032 0.035; visual mesh filename=file://robotis_op_description/meshes/arm_high_r.STL scale=1 1 1
- link MP_BODY: geometry collision box size=0.102 0.109 0.106; visual mesh filename=file://robotis_op_description/meshes/body.STL scale=1 1 1
- link MP_HEAD: geometry collision sphere radius=0.044; visual mesh filename=file://robotis_op_description/meshes/head.STL scale=1 1 1
- link MP_NECK: geometry collision box size=0.045 0.022 0.0325; visual mesh filename=file://robotis_op_description/meshes/neck.STL scale=1 1 1
- link MP_PELVIS_L: geometry collision box size=0.045 0.08175 0.028652; visual mesh filename=file://robotis_op_description/meshes/pelvis_l.STL scale=1 1 1
- link MP_PELVIS_R: geometry collision box size=0.045 0.08175 0.028652; visual mesh filename=file://robotis_op_description/meshes/pelvis_r.STL scale=1 1 1
- link MP_SHOULDER_L: geometry collision box size=0.016 0.033 0.02165; visual mesh filename=file://robotis_op_description/meshes/shoulder_l.STL scale=1 1 1
- link MP_SHOULDER_R: geometry collision box size=0.016 0.033 0.02165; visual mesh filename=file://robotis_op_description/meshes/shoulder_r.STL scale=1 1 1
- link MP_THIGH1_L: geometry collision box size=0.001 0.001 0.001; visual mesh filename=file://robotis_op_description/meshes/thigh1_l.STL scale=1 1 1
- link MP_THIGH1_R: geometry collision box size=0.001 0.001 0.001; visual mesh filename=file://robotis_op_description/meshes/thigh1_r.STL scale=1 1 1
- link MP_THIGH2_L: geometry collision box size=0.093 0.035 0.045; visual mesh filename=file://robotis_op_description/meshes/thigh2_l.STL scale=1 1 1
- link MP_THIGH2_R: geometry collision box size=0.093 0.035 0.045; visual mesh filename=file://robotis_op_description/meshes/thigh2_r.STL scale=1 1 1
- link MP_TIBIA_L: geometry collision box size=0.093 0.035 0.045; visual mesh filename=file://robotis_op_description/meshes/tibia_l.STL scale=1 1 1
- link MP_TIBIA_R: geometry collision box size=0.093 0.035 0.045; visual mesh filename=file://robotis_op_description/meshes/tibia_r.STL scale=1 1 1

File: robotis_op_description/robots/robotis_op_orig.urdf (robot description, URDF)
Before this commit: robot robotis_op2, 31 links, 30 joints
Links:
- link MP_ANKLE1_L: geometry collision box size=0.028652 0.08175 0.045; visual mesh filename=file://robotis_op_description/meshes/ankle1_l.STL scale=1 1 1
- link MP_ANKLE1_R: geometry collision box size=0.028652 0.08175 0.045; visual mesh filename=file://robotis_op_description/meshes/ankle1_r.STL scale=1 1 1
- link MP_ANKLE2_L: geometry collision box size=0.008 0.066 0.104; visual mesh filename=file://robotis_op_description/meshes/ankle2_l.STL scale=1 1 1
- link MP_ANKLE2_R: geometry collision box size=0.008 0.066 0.104; visual mesh filename=file://robotis_op_description/meshes/ankle2_r.STL scale=1 1 1
- link MP_ARM_HIGH_L: geometry collision box size=0.06 0.032 0.035; visual mesh filename=file://robotis_op_description/meshes/arm_high_l.STL scale=1 1 1
- link MP_ARM_HIGH_R: geometry collision box size=0.06 0.032 0.035; visual mesh filename=file://robotis_op_description/meshes/arm_high_r.STL scale=1 1 1
- link MP_BODY: geometry collision box size=0.102 0.109 0.106; visual mesh filename=file://robotis_op_description/meshes/body.STL scale=1 1 1
- link MP_HEAD: geometry collision sphere radius=0.044; visual mesh filename=file://robotis_op_description/meshes/head.STL scale=1 1 1
- link MP_NECK: geometry collision box size=0.045 0.022 0.0325; visual mesh filename=file://robotis_op_description/meshes/neck.STL scale=1 1 1
- link MP_PELVIS_L: geometry collision box size=0.045 0.08175 0.028652; visual mesh filename=file://robotis_op_description/meshes/pelvis_l.STL scale=1 1 1
- link MP_PELVIS_R: geometry collision box size=0.045 0.08175 0.028652; visual mesh filename=file://robotis_op_description/meshes/pelvis_r.STL scale=1 1 1
- link MP_SHOULDER_L: geometry collision box size=0.016 0.033 0.02165; visual mesh filename=file://robotis_op_description/meshes/shoulder_l.STL scale=1 1 1
- link MP_SHOULDER_R: geometry collision box size=0.016 0.033 0.02165; visual mesh filename=file://robotis_op_description/meshes/shoulder_r.STL scale=1 1 1
- link MP_THIGH1_L: geometry collision box size=0.001 0.001 0.001; visual mesh filename=file://robotis_op_description/meshes/thigh1_l.STL scale=1 1 1
- link MP_THIGH1_R: geometry collision box size=0.001 0.001 0.001; visual mesh filename=file://robotis_op_description/meshes/thigh1_r.STL scale=1 1 1
- link MP_THIGH2_L: geometry collision box size=0.093 0.035 0.045; visual mesh filename=file://robotis_op_description/meshes/thigh2_l.STL scale=1 1 1
- link MP_THIGH2_R: geometry collision box size=0.093 0.035 0.045; visual mesh filename=file://robotis_op_description/meshes/thigh2_r.STL scale=1 1 1
- link MP_TIBIA_L: geometry collision box size=0.093 0.035 0.045; visual mesh filename=file://robotis_op_description/meshes/tibia_l.STL scale=1 1 1
- link MP_TIBIA_R: geometry collision box size=0.093 0.035 0.045; visual mesh filename=file://robotis_op_description/meshes/tibia_r.STL scale=1 1 1

Commit message: Improve compatibility

File: robotis_op_description/robots/robotis_op_norm.urdf (robot description, URDF)
Before this commit: robot robotis_op2, 31 links, 30 joints
Links:
- link MP_ANKLE1_L: geometry collision box size=0.028652 0.08175 0.045; visual mesh filename=model://robotis_op_description/meshes/ankle1_l.STL scale=1 1 1
- link MP_ANKLE1_R: geometry collision box size=0.028652 0.08175 0.045; visual mesh filename=model://robotis_op_description/meshes/ankle1_r.STL scale=1 1 1
- link MP_ANKLE2_L: geometry collision box size=0.008 0.066 0.104; visual mesh filename=model://robotis_op_description/meshes/ankle2_l.STL scale=1 1 1
- link MP_ANKLE2_R: geometry collision box size=0.008 0.066 0.104; visual mesh filename=model://robotis_op_description/meshes/ankle2_r.STL scale=1 1 1
- link MP_ARM_HIGH_L: geometry collision box size=0.06 0.032 0.035; visual mesh filename=model://robotis_op_description/meshes/arm_high_l.STL scale=1 1 1
- link MP_ARM_HIGH_R: geometry collision box size=0.06 0.032 0.035; visual mesh filename=model://robotis_op_description/meshes/arm_high_r.STL scale=1 1 1
- link MP_BODY: geometry collision box size=0.102 0.109 0.106; visual mesh filename=model://robotis_op_description/meshes/body.STL scale=1 1 1
- link MP_HEAD: geometry collision sphere radius=0.044; visual mesh filename=model://robotis_op_description/meshes/head.STL scale=1 1 1
- link MP_NECK: geometry collision box size=0.045 0.022 0.0325; visual mesh filename=model://robotis_op_description/meshes/neck.STL scale=1 1 1
- link MP_PELVIS_L: geometry collision box size=0.045 0.08175 0.028652; visual mesh filename=model://robotis_op_description/meshes/pelvis_l.STL scale=1 1 1
- link MP_PELVIS_R: geometry collision box size=0.045 0.08175 0.028652; visual mesh filename=model://robotis_op_description/meshes/pelvis_r.STL scale=1 1 1
- link MP_SHOULDER_L: geometry collision box size=0.016 0.033 0.02165; visual mesh filename=model://robotis_op_description/meshes/shoulder_l.STL scale=1 1 1
- link MP_SHOULDER_R: geometry collision box size=0.016 0.033 0.02165; visual mesh filename=model://robotis_op_description/meshes/shoulder_r.STL scale=1 1 1
- link MP_THIGH1_L: geometry collision box size=0.001 0.001 0.001; visual mesh filename=model://robotis_op_description/meshes/thigh1_l.STL scale=1 1 1
- link MP_THIGH1_R: geometry collision box size=0.001 0.001 0.001; visual mesh filename=model://robotis_op_description/meshes/thigh1_r.STL scale=1 1 1
- link MP_THIGH2_L: geometry collision box size=0.093 0.035 0.045; visual mesh filename=model://robotis_op_description/meshes/thigh2_l.STL scale=1 1 1
- link MP_THIGH2_R: geometry collision box size=0.093 0.035 0.045; visual mesh filename=model://robotis_op_description/meshes/thigh2_r.STL scale=1 1 1
- link MP_TIBIA_L: geometry collision box size=0.093 0.035 0.045; visual mesh filename=model://robotis_op_description/meshes/tibia_l.STL scale=1 1 1
- link MP_TIBIA_R: geometry collision box size=0.093 0.035 0.045; visual mesh filename=model://robotis_op_description/meshes/tibia_r.STL scale=1 1 1

File: robotis_op_description/robots/robotis_op_orig.urdf (robot description, URDF)
Before this commit: robot robotis_op2, 31 links, 30 joints
Links:
- link MP_ANKLE1_L: geometry collision box size=0.028652 0.08175 0.045; visual mesh filename=model://robotis_op_description/meshes/ankle1_l.STL scale=1 1 1
- link MP_ANKLE1_R: geometry collision box size=0.028652 0.08175 0.045; visual mesh filename=model://robotis_op_description/meshes/ankle1_r.STL scale=1 1 1
- link MP_ANKLE2_L: geometry collision box size=0.008 0.066 0.104; visual mesh filename=model://robotis_op_description/meshes/ankle2_l.STL scale=1 1 1
- link MP_ANKLE2_R: geometry collision box size=0.008 0.066 0.104; visual mesh filename=model://robotis_op_description/meshes/ankle2_r.STL scale=1 1 1
- link MP_ARM_HIGH_L: geometry collision box size=0.06 0.032 0.035; visual mesh filename=model://robotis_op_description/meshes/arm_high_l.STL scale=1 1 1
- link MP_ARM_HIGH_R: geometry collision box size=0.06 0.032 0.035; visual mesh filename=model://robotis_op_description/meshes/arm_high_r.STL scale=1 1 1
- link MP_BODY: geometry collision box size=0.102 0.109 0.106; visual mesh filename=model://robotis_op_description/meshes/body.STL scale=1 1 1
- link MP_HEAD: geometry collision sphere radius=0.044; visual mesh filename=model://robotis_op_description/meshes/head.STL scale=1 1 1
- link MP_NECK: geometry collision box size=0.045 0.022 0.0325; visual mesh filename=model://robotis_op_description/meshes/neck.STL scale=1 1 1
- link MP_PELVIS_L: geometry collision box size=0.045 0.08175 0.028652; visual mesh filename=model://robotis_op_description/meshes/pelvis_l.STL scale=1 1 1
- link MP_PELVIS_R: geometry collision box size=0.045 0.08175 0.028652; visual mesh filename=model://robotis_op_description/meshes/pelvis_r.STL scale=1 1 1
- link MP_SHOULDER_L: geometry collision box size=0.016 0.033 0.02165; visual mesh filename=model://robotis_op_description/meshes/shoulder_l.STL scale=1 1 1
- link MP_SHOULDER_R: geometry collision box size=0.016 0.033 0.02165; visual mesh filename=model://robotis_op_description/meshes/shoulder_r.STL scale=1 1 1
- link MP_THIGH1_L: geometry collision box size=0.001 0.001 0.001; visual mesh filename=model://robotis_op_description/meshes/thigh1_l.STL scale=1 1 1
- link MP_THIGH1_R: geometry collision box size=0.001 0.001 0.001; visual mesh filename=model://robotis_op_description/meshes/thigh1_r.STL scale=1 1 1
- link MP_THIGH2_L: geometry collision box size=0.093 0.035 0.045; visual mesh filename=model://robotis_op_description/meshes/thigh2_l.STL scale=1 1 1
- link MP_THIGH2_R: geometry collision box size=0.093 0.035 0.045; visual mesh filename=model://robotis_op_description/meshes/thigh2_r.STL scale=1 1 1
- link MP_TIBIA_L: geometry collision box size=0.093 0.035 0.045; visual mesh filename=model://robotis_op_description/meshes/tibia_l.STL scale=1 1 1
- link MP_TIBIA_R: geometry collision box size=0.093 0.035 0.045; visual mesh filename=model://robotis_op_description/meshes/tibia_r.STL scale=1 1 1
