Commit message: repair model

File: robotis_op_description/urdf/torso/robotis_op_torso.urdf.xacro (robot description, xacro)
@@ -8,5 +8,5 @@
       <origin xyz="-0.003053 -0.038651 -0.019268" />
       <mass value="0.97559947"/>
-      <inertia ixx="0.001879411079" ixy="0.0" ixz="0.0" iyy="0.00175933104423" iyz="0.0" izz="0.00181176951575"/>
+      <inertia ixx="3.1081800"  ixy="-0.25460189"  ixz="2.0318174" iyy="6.3787776" iyz="0.16417863" izz="5.3316425" />
     </inertial>
     <body_collision_geom_macro />
